File: hardware/RK3399_PIKVM/RK3399_PIKVM.kicad_sch (KiCad schematic)
At the start: 5 parts, among them U1 RK3399

Commit message: Updated schematics.
Other:
- note added: "DDR3 2GB SRAM"
- note added: "PCIE & M.2 Port"
- note added: "Power Ground and Power VDD"
- note added: "RK3399 DDR0 Port"
- note added: "RK3399 DDR1 Port"
- moved on the sheet: U1A, U1B, U1C, U1D, U1E, U1F, U1G, U1H, U1I, U1J, U1K, U1L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

Commit message: Updated schematic.
Parts:
- added U6: ~, symbol zgoolib:RK808D
Other:
- note added: "16GB eMMC"
- note added: "A53 Power"
- note added: "A72 Power"
- note added: "BOOT Media"
- note added: "GPIO PINs"
- note added: "GPU Power"
- note added: "HDMI Input"
- note added: "HDMI Output"
- note added: "ISP & UART"
- note added: "Other LDOs"
- note added: "Power Manage IC"
- note added: "RK3399 PiKVM"
- note added: "SD Card"
- note added: "USB2 & USB3"
- moved on the sheet: U1A, U1B, U1D, U1E, U1F, U1H, U1K, U1L, U1M, U1N, U1O, U1P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

Commit message: Finished the function allocation.
Other:
- note added: "Ethernet Port"
- moved on the sheet: U1A, U1B, U1D, U1E, U1F, U1M, U1Q, U1S, U1T, U1W, U1X, U1Z
