File: hardware/RK3399_PIKVM/RK3399_PIKVM.kicad_sch (KiCad schematic)
At the start: 6 parts, among them U1 RK3399

Commit message: Updated schematic
Parts:
- removed U2, U3: ~, Package_BGA:BGA-96_9.0x13.0mm_Layout2x3x16_P0.8mm, symbol zgoolib:H5TQ4G63AFR
- added POWER1: DC-05-SMD-Connector, symbol zgoolib:DC-05-SMD-Connector
- added R1, R2, R3, R4, R5, R6, R7, R8: 0402 240Ω/1%, symbol Device:R_Small
- added U4, U5: ~, Package_BGA:BGA-96_9.0x13.0mm_Layout2x3x16_P0.8mm, symbol zgoolib:H5TQ4G63AFR
- U1: footprint BGA828C65P31X31_2100X2100X161N -> zgoolib:RK3399
- U6: footprint (none) -> Package_DFN_QFN:QFN-68-1EP_8x8mm_P0.4mm_EP5.2x5.2mm
- renumbered U4 to U2, U5 to U3
Connections:
- net VSS: now reaches U3.A9 (VSS#9)
- net VSS: now also U1.A1 (VSS_1), U1.A27 (VSS_2), U1.A31 (VSS_3), U1.AA10 (VSS_179), U1.AA11 (AVSS_13), U1.AA12 (AVSS_17), U1.AA13 (VSS_177), U1.AA14 (AVSS_26), U1.AA15 (AVSS_53), U1.AA23 (AVSS_4), U1.AA26 (AVSS_6), U1.AA29 (AVSS_7), U1.AA3 (VSS_4), U1.AA5 (VSS_5), U1.AA9 (VSS_6), U1.AB10 (AVSS_12), U1.AB11 (AVSS_8), U1.AB13 (AVSS_9), U1.AB15 (AVSS_42), U1.AB16 (AVSS_41), U1.AB17 (AVSS_52), U1.AB19 (VSS_140), U1.AB23 (AVSS_5), U1.AB9 (VSS_9), U1.AC11 (AVSS_44), U1.AC13 (AVSS_45), U1.AC15 (AVSS_10), U1.AC16 (AVSS_18), U1.AC17 (AVSS_43), U1.AC18 (VSS_145), U1.AC20 (VSS_13), U1.AC21 (VSS_132), U1.AC22 (VSS_12), U1.AC23 (AVSS_19), U1.AC25 (AVSS_51), U1.AC26 (AVSS_14), U1.AC29 (AVSS_15), U1.AC3 (VSS_16), U1.AD10 (VSS_19), U1.AD13 (AVSS_11), U1.AD17 (AVSS_16), U1.AD21 (VSS_163), U1.AD22 (VSS_11), U1.AD26 (AVSS_40), U1.AD29 (AVSS_20), U1.AD3 (VSS_17), U1.AD5 (VSS_18), U1.AE11 (AVSS_21), U1.AE12 (AVSS_22), U1.AE14 (AVSS_23), U1.AE17 (AVSS_24), U1.AE23 (VSS_14), U1.AE27 (AVSS_25), U1.AF17 (AVSS_27), U1.AF18 (VSS_7), U1.AF20 (VSS_10), U1.AF23 (AVSS_2), U1.AF24 (AVSS_3), U1.AF29 (AVSS_28), U1.AF9 (VSS_20), U1.AG2 (VSS_21), U1.AG29 (AVSS_29), U1.AH29 (AVSS_30), U1.AJ11 (AVSS_34), U1.AJ12 (AVSS_35), U1.AJ14 (AVSS_36), U1.AJ15 (AVSS_37), U1.AJ17 (AVSS_38), U1.AJ18 (AVSS_39), U1.AJ20 (VSS_180), U1.AJ21 (VSS_172), U1.AJ23 (VSS_173), U1.AJ24 (VSS_174), U1.AJ26 (VSS_175), U1.AJ27 (VSS_176), U1.AJ28 (VSS_171), U1.AJ29 (AVSS_47), U1.AJ5 (VSS_22), U1.AJ6 (AVSS_31), U1.AJ8 (AVSS_32), U1.AJ9 (AVSS_33), U1.AL1 (VSS_23), U1.AL31 (VSS_178), U1.B5 (VSS_24), U1.C11 (VSS_27), U1.C12 (VSS_28), U1.C14 (VSS_29), U1.C15 (VSS_30), U1.C17 (VSS_31), U1.C18 (VSS_32), U1.C20 (VSS_33), U1.C21 (VSS_34), U1.C23 (VSS_35), U1.C24 (VSS_36), U1.C26 (VSS_37), U1.C8 (VSS_25), U1.C9 (VSS_26), U1.D5 (VSS_38), U1.E12 (VSS_42), U1.E15 (VSS_43), U1.E18 (VSS_44), U1.E2 (VSS_39), U1.E21 (VSS_45), U1.E24 (VSS_46), U1.E31 (VSS_47), U1.E4 (VSS_40), U1.E7 (VSS_41), U1.F15 (VSS_49), U1.F18 (VSS_50), U1.F20 (VSS_51), U1.F21 (VSS_52), U1.F8 (VSS_48), U1.G18 (VSS_55), U1.G27 (VSS_56), U1.G5 (VSS_53), U1.G9 (VSS_54), U1.H10 (VSS_59), U1.H11 (VSS_60), U1.H12 (VSS_61), U1.H13 (VSS_62), U1.H15 (VSS_63), U1.H16 (VSS_64), U1.H17 (VSS_65), U1.H18 (VSS_66), U1.H26 (VSS_67), U1.H3 (VSS_57), U1.H9 (VSS_58), U1.J10 (VSS_73), U1.J3 (VSS_68), U1.J6 (VSS_69), U1.J7 (VSS_70), U1.J8 (VSS_71), U1.J9 (VSS_72), U1.K10 (VSS_76), U1.K12 (VSS_77), U1.K14 (VSS_78), U1.K16 (VSS_79), U1.K18 (VSS_80), U1.K20 (VSS_82), U1.K22 (VSS_84), U1.K8 (VSS_74), U1.K9 (VSS_75), U1.L11 (VSS_88), U1.L12 (VSS_89), U1.L13 (VSS_90), U1.L14 (VSS_91), U1.L15 (VSS_92), U1.L16 (VSS_93), U1.L20 (VSS_96), U1.L22 (VSS_97), U1.L27 (VSS_99), U1.L3 (VSS_85), U1.L6 (VSS_86), U1.L8 (VSS_87), U1.M10 (VSS_102), U1.M16 (VSS_103), U1.M23 (VSS_104), U1.M3 (VSS_100), U1.M8 (VSS_101), U1.N13 (VSS_108), U1.N14 (VSS_109), U1.N15 (VSS_110), U1.N16 (VSS_111), U1.N17 (VSS_94), U1.N19 (VSS_83), U1.N21 (VSS_98), U1.N8 (VSS_105), U1.P10 (VSS_116), U1.P11 (VSS_106), U1.P12 (VSS_107), U1.P16 (VSS_117), U1.P19 (VSS_119), U1.P21 (VSS_121), U1.P3 (VSS_112), U1.P6 (VSS_113), U1.P7 (VSS_114), U1.P8 (VSS_115), U1.R14 (VSS_129), U1.R15 (VSS_130), U1.R16 (VSS_131), U1.R18 (VSS_165), U1.R21 (VSS_120), U1.R23 (VSS_133), U1.R3 (VSS_123), U1.R5 (VSS_124), U1.R6 (VSS_125), U1.T10 (VSS_135), U1.T16 (VSS_138), U1.T18 (VSS_168), U1.T19 (VSS_122), U1.T21 (VSS_139), U1.T8 (VSS_134), U1.U11 (VSS_126), U1.U12 (VSS_127), U1.U14 (VSS_137), U1.U15 (VSS_143), U1.U16 (VSS_144), U1.U19 (VSS_146), U1.U21 (VSS_147), U1.U22 (VSS_149), U1.U23 (AVSS_49), U1.U29 (VSS_150), U1.U3 (VSS_141), U1.U8 (VSS_142), U1.V10 (VSS_154), U1.V17 (VSS_148), U1.V23 (AVSS_50), U1.V3 (VSS_151), U1.V5 (VSS_152), U1.V8 (VSS_153), U1.W13 (VSS_128), U1.W17 (VSS_159), U1.W18 (VSS_169), U1.W19 (VSS_167), U1.W21 (VSS_81), U1.W22 (VSS_158), U1.W23 (AVSS_46), U1.W30 (VSS_160), U1.W8 (VSS_161), U1.W9 (VSS_162), U1.Y10 (VSS_15), U1.Y11 (VSS_155), U1.Y12 (VSS_136), U1.Y13 (VSS_164), U1.Y14 (VSS_156), U1.Y15 (VSS_157), U1.Y16 (VSS_118), U1.Y17 (VSS_95), U1.Y20 (VSS_170), U1.Y23 (AVSS_1), U1.Y29 (AVSS_48), U1.Y3 (VSS_8), U1.Y9 (VSS_166), U2.A9 (VSS#9), U2.B1 (VSSQ#1), U2.B3 (VSS#6), U2.B9 (VSSQ#7), U2.D1 (VSSQ#2), U2.D8 (VSSQ#5), U2.E1 (VSS#1), U2.E2 (VSSQ#4), U2.E8 (VSSQ#6), U2.F9 (VSSQ#8), U2.G1 (VSSQ#3), U2.G8 (VSS#7), U2.G9 (VSSQ#9), U2.J2 (VSS#5), U2.J8 (VSS#8), U2.M1 (VSS#2), U2.M9 (VSS#10), U2.P1 (VSS#3), U2.P9 (VSS#11), U2.T1 (VSS#4), U2.T9 (VSS#12), U3.B1 (VSSQ#1), U3.B3 (VSS#6), U3.B9 (VSSQ#7), U3.D1 (VSSQ#2), U3.D8 (VSSQ#5), U3.E1 (VSS#1), U3.E2 (VSSQ#4), U3.E8 (VSSQ#6), U3.F9 (VSSQ#8), U3.G1 (VSSQ#3), U3.G8 (VSS#7), U3.G9 (VSSQ#9), U3.J2 (VSS#5), U3.J8 (VSS#8), U3.M1 (VSS#2), U3.M9 (VSS#10), U3.P1 (VSS#3), U3.P9 (VSS#11), U3.T1 (VSS#4), U3.T9 (VSS#12), R1.2, R2.2, R3.2, R4.2, R5.2, R6.2, R7.2, R8.2, U4.A9 (VSS#9), U4.B1 (VSSQ#1), U4.B3 (VSS#6), U4.B9 (VSSQ#7), U4.D1 (VSSQ#2), U4.D8 (VSSQ#5), U4.E1 (VSS#1), U4.E2 (VSSQ#4), U4.E8 (VSSQ#6), U4.F9 (VSSQ#8), U4.G1 (VSSQ#3), U4.G8 (VSS#7), U4.G9 (VSSQ#9), U4.J2 (VSS#5), U4.J8 (VSS#8), U4.M1 (VSS#2), U4.M9 (VSS#10), U4.P1 (VSS#3), U4.P9 (VSS#11), U4.T1 (VSS#4), U4.T9 (VSS#12), U5.A9 (VSS#9), U5.B1 (VSSQ#1), U5.B3 (VSS#6), U5.B9 (VSSQ#7), U5.D1 (VSSQ#2), U5.D8 (VSSQ#5), U5.E1 (VSS#1), U5.E2 (VSSQ#4), U5.E8 (VSSQ#6), U5.F9 (VSSQ#8), U5.G1 (VSSQ#3), U5.G8 (VSS#7), U5.G9 (VSSQ#9), U5.J2 (VSS#5), U5.J8 (VSS#8), U5.M1 (VSS#2), U5.M9 (VSS#10), U5.P1 (VSS#3), U5.P9 (VSS#11), U5.T1 (VSS#4), U5.T9 (VSS#12)
- net DDR0_A10: now reaches U3.L7 (A10)
- net DDR0_A10: now also U1.D1 (DDR0_A10), U2.L7 (A10)
- net at U3.L8 (ZQ): now also R8.1
- net at U3.L9 (ZQ1): now also R7.1
- net DDR0_BA0: now reaches U3.M2 (BA0)
- net DDR0_BA0: now also U1.C3 (DDR0_BA0), U2.M2 (BA0)
- net DDR0_BA2: now reaches U3.M3 (BA2)
- net DDR0_BA2: now also U1.M4 (DDR0_BA2), U2.M3 (BA2)
- net DDR0_A15: now reaches U3.M7 (A15)
- net DDR0_A15: now also U1.H7 (DDR0_A15), U2.M7 (A15)
- net DDR0_A3: now reaches U3.N2 (A3)
- net DDR0_A3: now also U1.G2 (DDR0_A3), U2.N2 (A3)
- net DDR0_A0: now reaches U3.N3 (A0)
- net DDR0_A0: now also U1.F2 (DDR0_A0), U2.N3 (A0)
- net DDR0_A12: now reaches U3.N7 (A12)
- net DDR0_A12: now also U1.C1 (DDR0_A12), U2.N7 (A12)
- net DDR0_BA1: now reaches U3.N8 (BA1)
- net DDR0_BA1: now also U1.F4 (DDR0_BA1), U2.N8 (BA1)
- net DDR0_A5: now reaches U3.P2 (A5)
- net DDR0_A5: now also U1.H1 (DDR0_A5), U2.P2 (A5)
- net DDR0_A2: now reaches U3.P3 (A2)
- net DDR0_A2: now also U1.G1 (DDR0_A2), U2.P3 (A2)
- net DDR0_A1: now reaches U3.P7 (A1)
- net DDR0_A1: now also U1.F1 (DDR0_A1), U2.P7 (A1)
- net DDR0_A4: now reaches U3.P8 (A4)
- net DDR0_A4: now also U1.H2 (DDR0_A4), U2.P8 (A4)
- net DDR0_A7: now reaches U3.R2 (A7)
- net DDR0_A7: now also U1.J2 (DDR0_A7), U2.R2 (A7)
- net DDR0_A9: now reaches U3.R3 (A9)
- net DDR0_A9: now also U1.K1 (DDR0_A9), U2.R3 (A9)
- net DDR0_A11: now reaches U3.R7 (A11)
- net DDR0_A11: now also U1.E3 (DDR0_A11), U2.R7 (A11)
- net DDR0_A6: now reaches U3.R8 (A6)
- net DDR0_A6: now also U1.J1 (DDR0_A6), U2.R8 (A6)
- net DDR0_A13: now reaches U3.T3 (A13)
- net DDR0_A13: now also U1.D2 (DDR0_A13), U2.T3 (A13)
- net DDR0_A14: now reaches U3.T7 (A14)
- net DDR0_A14: now also U1.D3 (DDR0_A14), U2.T7 (A14)
- net DDR0_A8: now reaches U3.T8 (A8)
- net DDR0_A8: now also U1.K2 (DDR0_A8), U2.T8 (A8)
- net at U2.L8 (ZQ): now also R6.1
- net at U2.L9 (ZQ1): now also R5.1
- net at U1.L10 (DDR0_VDD_2): now also U1.L9 (DDR0_VDD_1), U1.M9 (DDR0_VDD_3), U1.N10 (DDR0_VDD_5), U1.N9 (DDR0_VDD_4), U1.P9 (DDR0_VDD_6), U1.R9 (DDR0_VDD_7)
- net at U1.R10 (DDR0_VDD_8): now also U1.T9 (DDR0_VDD_9), U1.U10 (DDR0_VDD_11), U1.U9 (DDR0_VDD_10), U1.V9 (DDR0_VDD_12)
- net DDR1_A1: now reaches U1.A10 (DDR1_A1)
- net DDR1_A1: now also U4.P7 (A1), U5.P7 (A1)
- net DDR1_A12: now reaches U1.A3 (DDR1_A12)
- net DDR1_A12: now also U4.N7 (A12), U5.N7 (A12)
- net DDR1_A10: now reaches U1.A4 (DDR1_A10)
- net DDR1_A10: now also U4.L7 (A10), U5.L7 (A10)
- net DDR1_A9: now reaches U1.A6 (DDR1_A9)
- net DDR1_A9: now also U4.R3 (A9), U5.R3 (A9)
- net DDR1_A7: now reaches U1.A7 (DDR1_A7)
- net DDR1_A7: now also U4.R2 (A7), U5.R2 (A7)
- net DDR1_A5: now reaches U1.A8 (DDR1_A5)
- net DDR1_A5: now also U4.P2 (A5), U5.P2 (A5)
- net DDR1_A3: now reaches U1.A9 (DDR1_A3)
- net DDR1_A3: now also U4.N2 (A3), U5.N2 (A3)
- net DDR1_A0: now reaches U1.B10 (DDR1_A0)
- net DDR1_A0: now also U4.N3 (A0), U5.N3 (A0)
- net DDR1_BA0: now reaches U1.B2 (DDR1_BA0)
- net DDR1_BA0: now also U4.M2 (BA0), U5.M2 (BA0)
- net DDR1_A13: now reaches U1.B4 (DDR1_A13)
- net DDR1_A13: now also U4.T3 (A13), U5.T3 (A13)
- net DDR1_A8: now reaches U1.B6 (DDR1_A8)
- net DDR1_A8: now also U4.T8 (A8), U5.T8 (A8)
- net DDR1_A6: now reaches U1.B7 (DDR1_A6)
- net DDR1_A6: now also U4.R8 (A6), U5.R8 (A6)
- net DDR1_A4: now reaches U1.B8 (DDR1_A4)
- net DDR1_A4: now also U4.P8 (A4), U5.P8 (A4)
- net DDR1_A2: now reaches U1.B9 (DDR1_A2)
- net DDR1_A2: now also U4.P3 (A2), U5.P3 (A2)
- net DDR1_A14: now reaches U1.C4 (DDR1_A14)
- net DDR1_A14: now also U4.T7 (A14), U5.T7 (A14)
- net DDR1_A11: now reaches U1.C5 (DDR1_A11)
- net DDR1_A11: now also U4.R7 (A11), U5.R7 (A11)
- net DDR1_BA2: now reaches U1.D12 (DDR1_BA2)
- net DDR1_BA2: now also U4.M3 (BA2), U5.M3 (BA2)
- net DDR1_BA1: now reaches U1.D6 (DDR1_BA1)
- net DDR1_BA1: now also U4.N8 (BA1), U5.N8 (BA1)
- net DDR1_A15: now reaches U1.G8 (DDR1_A15)
- net DDR1_A15: now also U4.M7 (A15), U5.M7 (A15)
- net at U1.J11 (DDR1_VDD_1): now also U1.J12 (DDR1_VDD_2), U1.J13 (DDR1_VDD_3), U1.J14 (DDR1_VDD_4), U1.J15 (DDR1_VDD_5), U1.J16 (DDR1_VDD_6), U1.J17 (DDR1_VDD_7)
- net at U1.J18 (DDR1_VDD_8): now also U1.K11 (DDR1_VDD_9), U1.K13 (DDR1_VDD_10), U1.K15 (DDR1_VDD_11), U1.K17 (DDR1_VDD_12)
- new net: R2.1, U5.L8 (ZQ)
- new net: R1.1, U5.L9 (ZQ1)
- new net: R4.1, U4.L8 (ZQ)
- new net: R3.1, U4.L9 (ZQ1)
- now unconnected: U1.AA19 (NC), U1.AA20 (NC), U1.AA22 (NC), U1.AB20 (NC), U1.AB22 (NC), U1.AC12 (NC), U1.AC14 (NC), U1.AD11 (NC), U1.AD12 (NC), U1.AD14 (NC), U1.AD15 (NC)
Other:
- note added: "1. PowerManage IC"
- note added: "2. RK3399 Power Input"
- note added: "3. DDR"
- note added: "DC-05 Port"
- note added: "DDR0 Addr"
- note added: "DDR0 High 16bits"
- note added: "DDR0 Low 16bits"
- note added: "DDR1 Addr"
- note added: "DDR1 High 16bits"
- note added: "DDR1 Low 16bits"
- note removed: "Other LDOs"
- moved on the sheet: U1A, U1B, U1C, U1D, U1E, U1F, U1G, U1I, U1J, U2, U3

Commit message: Updated schematic.
Parts:
- added U7: TPS54821RHLR, zgoolib:TPS54821, symbol zgoolib:TPS54821RHLR
- added U8: RTL8211F-CG, zgoolib:RTL8188_QFN40, symbol zgoolib:RTL8211F-CG
Connections:
- net at U3.B2 (VDD#3): now also U3.D9 (VDD#7), U3.G7 (VDD#5), U3.K2 (VDD#4), U3.K8 (VDD#6), U3.N1 (VDD#1), U3.N9 (VDD#8), U3.R1 (VDD#2), U3.R9 (VDD#9)
- net at U2.B2 (VDD#3): now also U2.D9 (VDD#7), U2.G7 (VDD#5), U2.K2 (VDD#4), U2.K8 (VDD#6), U2.N1 (VDD#1), U2.N9 (VDD#8), U2.R1 (VDD#2), U2.R9 (VDD#9)
- net at U5.A1 (VDDQ#1): now also U5.A8 (VDDQ#6), U5.C1 (VDDQ#2), U5.C9 (VDDQ#9), U5.D2 (VDDQ#4), U5.E9 (VDDQ#8), U5.F1 (VDDQ#3), U5.H2 (VDDQ#5), U5.H9 (VDDQ#7)
- net at U5.B2 (VDD#3): now also U5.D9 (VDD#7), U5.G7 (VDD#5), U5.K2 (VDD#4), U5.K8 (VDD#6), U5.N1 (VDD#1), U5.N9 (VDD#8), U5.R1 (VDD#2), U5.R9 (VDD#9)
- net at U4.A1 (VDDQ#1): now also U4.A8 (VDDQ#6), U4.C1 (VDDQ#2), U4.C9 (VDDQ#9), U4.D2 (VDDQ#4), U4.E9 (VDDQ#8), U4.F1 (VDDQ#3), U4.H2 (VDDQ#5), U4.H9 (VDDQ#7)
- net at U4.B2 (VDD#3): now also U4.D9 (VDD#7), U4.G7 (VDD#5), U4.K2 (VDD#4), U4.K8 (VDD#6), U4.N1 (VDD#1), U4.N9 (VDD#8), U4.R1 (VDD#2), U4.R9 (VDD#9)
Other:
- note added: "1000M Ethernet Port"
- note removed: "Ethernet Port"
- moved on the sheet: POWER1, U1C, U1O, U1X, U6

Commit message: Updated some datasheets and ref PDFs
Parts:
- added U10: SR9900A, Package_DFN_QFN:QFN-24-1EP_4x4mm_P0.5mm_EP2.6x2.6mm, symbol zgoolib:SR9900
Other:
- moved on the sheet: U1H
Changed lines of the file:
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@@
     (effects (font (size 8 8) (thickness 1.6) bold (color 132 0 0 1)) (justify right bottom))
   )
-  (text "PCIE & M.2 Port" (at 492.506 739.394 0)
+  (text "PCIE & M.2 Port" (at 426.72 704.85 0)
     (effects (font (size 8 8) (thickness 1.6) bold (color 132 0 0 1)) (justify right bottom))
   )
@@
     )
   )
-  (symbol (lib_id "RK3399:RK3399") (at 444.5 782.32 0) (unit 8)
+  (symbol (lib_id "RK3399:RK3399") (at 511.81 782.32 0) (unit 8)
     (in_bom yes) (on_board yes) (dnp no) (fields_autoplaced)
-    (property "Reference" "U1" (at 447.1871 753.11 0)
+    (property "Reference" "U1" (at 514.4971 753.11 0)
       (effects (font (size 1.27 1.27)))
     )
-    (property "Value" "RK3399" (at 447.1871 755.65 0)
+    (property "Value" "RK3399" (at 514.4971 755.65 0)
       (effects (font (size 1.27 1.27)))
     )
-    (property "Footprint" "zgoolib:RK3399" (at 444.5 904.24 0)
+    (property "Footprint" "zgoolib:RK3399" (at 511.81 904.24 0)
       (effects (font (size 1.27 1.27)) (justify bottom) hide)
     )
-    (property "Datasheet" "" (at 444.5 782.32 0)
+    (property "Datasheet" "" (at 511.81 782.32 0)
       (effects (font (size 1.27 1.27)) hide)
     )
-    (property "MF" "Rockchip" (at 444.5 901.7 0)
+    (property "MF" "Rockchip" (at 511.81 901.7 0)
       (effects (font (size 1.27 1.27)) (justify bottom) hide)
     )
-    (property "Description" "RK3399 ROCK Pi 4 Model A 2GB - ARM® Cortex®-A53, Cortex®-A72 MPU Embedded Evaluation Board" (at 444.5 916.94 0)
+    (property "Description" "RK3399 ROCK Pi 4 Model A 2GB - ARM® Cortex®-A53, Cortex®-A72 MPU Embedded Evaluation Board" (at 511.81 916.94 0)
       (effects (font (size 1.27 1.27)) (justify bottom) hide)
     )
-    (property "Package" "Seeed Technology" (at 444.5 906.78 0)
+    (property "Package" "Seeed Technology" (at 511.81 906.78 0)
       (effects (font (size 1.27 1.27)) (justify bottom) hide)
     )
-    (property "Price" "None" (at 444.5 909.32 0)
+    (property "Price" "None" (at 511.81 909.32 0)
       (effects (font (size 1.27 1.27)) (justify bottom) hide)
     )
-    (property "MP" "RK3399" (at 444.5 914.4 0)
+    (property "MP" "RK3399" (at 511.81 914.4 0)
       (effects (font (size 1.27 1.27)) (justify bottom) hide)
     )
-    (property "Availability" "Not in stock" (at 444.5 911.86 0)
+    (property "Availability" "Not in stock" (at 511.81 911.86 0)
       (effects (font (size 1.27 1.27)) (justify bottom) hide)
     )
@@
         )
       )
+    )
+  )
+  (symbol (lib_id "zgoolib:SR9900") (at 881.38 591.82 0) (unit 1)
+    (in_bom yes) (on_board yes) (dnp no)
+    (property "Reference" "U10" (at 864.87 570.23 0)
+      (effects (font (size 1.27 1.27)))
+    )
+    (property "Value" "SR9900A" (at 864.87 572.77 0)
+      (effects (font (size 1.27 1.27)))
+    )
+    (property "Footprint" "Package_DFN_QFN:QFN-24-1EP_4x4mm_P0.5mm_EP2.6x2.6mm" (at 881.38 624.84 0)
+      (effects (font (size 1.27 1.27)) (justify bottom) hide)
+    )
+    (property "Datasheet" "" (at 881.38 632.46 0)
+      (effects (font (size 1.27 1.27)) hide)
+    )
+    (pin "1")
+    (pin "10")
+    (pin "11")
+    (pin "12")
+    (pin "13")
+    (pin "14")
+    (pin "15")
+    (pin "16")
+    (pin "17")
+    (pin "18")
+    (pin "19")
+    (pin "2")
+    (pin "20")
+    (pin "21")
+    (pin "22")
+    (pin "23")
+    (pin "24")
+    (pin "3")
+    (pin "4")
+    (pin "5")
+    (pin "6")
+    (pin "7")
+    (pin "8")
+    (pin "9")
+    (pin "25")
+    (instances
+      (project "RK3399_PIKVM"
+        (path "/d1897343-8887-4fc7-b5d3-4f92f4433ed8"
+          (reference "U10") (unit 1)
+        )
+      )

Commit message: Updated schematic
Parts:
- removed U10: SR9900A, Package_DFN_QFN:QFN-24-1EP_4x4mm_P0.5mm_EP2.6x2.6mm, symbol zgoolib:SR9900
- added J1, J2: HR911105A, zgoolib:RJ45_HanRun_HR911105A, symbol zgoolib:HR911105A
- added U9: RTL8111H-CG, Package_DFN_QFN:QFN-32-1EP_4x4mm_P0.4mm_EP2.65x2.65mm, symbol zgoolib:RTL8111H-CG
Other:
- note added: "Dual 1000M Ethernet Port"
- note removed: "1000M Ethernet Port"
- moved on the sheet: U1B, U1D, U1E, U1F, U1M, U1Q, U1S, U1T, U1W, U1X, U1Z, U8
