File: hardware/RK3399_PIKVM/RK3399_PIKVM.kicad_sch (KiCad schematic)
At the start: 20 parts, among them J1 HR911105A, J2 HR911105A, U1 RK3399, U7 TPS54821RHLR, U8 RTL8211F-CG, U9 RTL8111H-CG

Commit message: Updated some contents
Parts:
- added SD1: ~, zgoolib:TF-SMD_TF-01A, symbol zgoolib:SD_Socket_SelfLock
- POWER1: footprint (none) -> zgoolib:DC-05_SMD
- U8: footprint zgoolib:RTL8188_QFN40 -> zgoolib:RTL8211_QFN40
Other:
- note added: "Used for control the power"
- moved on the sheet: R1, R2, R3, R4, R5, R6, R7, R8, U1A, U1I, U1J, U1L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
