File: hardware/RK3399_PIKVM/RK3399_PIKVM.kicad_pcb (KiCad board)
At the start: 6 copper layers, 100 x 100 mm, 15 parts, among them J1 HR911105A, J2 HR911105A, M3 M3_Whole, U1 RK3399, U7 TPS54821RHLR, U8 RTL8211F-CG, U9 RTL8111H-CG

Commit message: Updated some contents
Parts:
- added POWER1: DC-05-SMD-Connector, zgoolib:DC-05_SMD, F.Cu at (154.1, 59.6)
- added SD1: ~, zgoolib:TF-SMD_TF-01A, F.Cu at (80.4, 112.1)
- U8: footprint zgoolib:RTL8188_QFN40 -> zgoolib:RTL8211_QFN40
- moved U8 5.45 mm to (101.9, 96.5), turned to 0 degrees
